Commit message: update controoller

File: softleg_description/urdf/softleg_FC_fixedcart.urdf (robot description, URDF)
Before this commit: robot softlegisaac, 7 links, 6 joints
Joints:
- joint softleg_1_ankle_joint: limit lower=-3.1415927 upper=3.1415927 effort=11. velocity=100. -> lower=-3.1415927 upper=3.1415927 effort=150. velocity=100.
- joint softleg_1_cart_joint: origin xyz=0. 0.2102 0.  rpy=0.0 0.0 0.0  -> xyz=0. 0.60 0.  rpy=0.0 0.0 0.0 ; type prismatic -> fixed
- joint softleg_1_hip_joint: limit lower=-3.1415927 upper=3.1415927 effort=11. velocity=100. -> lower=-3.1415927 upper=3.1415927 effort=150. velocity=300.
- joint softleg_1_knee_joint: limit lower=-3.1415927 upper=3.1415927 effort=11. velocity=100. -> lower=-3.1415927 upper=3.1415927 effort=150. velocity=300.
